File: bob/bob.kicad_pcb (KiCad board)
At the start: 4 copper layers, 62 x 19 mm, 28 parts, among them J1 PROG, J2 PWR, J3 BB, U1 PAN2110P0AA, U2 LM1117MP-3.3, U3 PY32F030K1xTx, Y1 16MHz

Commit message: WIP
Parts:
- removed C1, C2, C3, C4: NC, Capacitor_SMD:C_0805_2012Metric
- removed R2: 0R, Resistor_SMD:R_0805_2012Metric
- added JP2: I2C/SPI, Jumper:SolderJumper-3_P2.0mm_Open_TrianglePad1.0x1.5mm, F.Cu at (232.0, 54.5)
- R1: value 0R -> 10k
- moved R1 9.39 mm to (233.5, 63.5), turned to 0 degrees
- moved Y1 2.00 mm to (239.5, 63.0)
- moved A1 1.12 mm to (239.0, 54.0)
- moved U1 1.12 mm to (233.5, 59.0)
Connections:
- J1 pad 3: /PROG_TXD -> /PROG_RXD
- J1 pad 5: /PROG_RXD -> /PROG_TXD
- R1 pad 1: Net-(U1-ANT) -> /~{RF_CS}
- R1 pad 2: Net-(A1-A) -> Net-(JP2-C)
- U1 pad 8: Net-(U1-ANT) -> Net-(A1-A)
- Y1 pad 1: Net-(C4-Pad2) -> Net-(U1-XC1)
Routing:
- net Net-(JP2-C): track 0.00 -> 10.00 mm
- net /~{RF_CS}: track 17.9 -> 26.6 mm
- net Net-(C4-Pad2): track 5.19 -> 0.00 mm
- net +3V3: track 25.0 -> 28.1 mm
- net /RF_CLK: track 23.1 -> 20.3 mm
- net Net-(U1-XC0): track 8.28 -> 5.67 mm
- net Net-(U1-XC1): track 2.46 -> 4.13 mm
- net /PROG_RXD: track 32.4 -> 33.7 mm
- net /RF_DIO: track 26.7 -> 25.6 mm
- net /PF3: track 26.3 -> 25.2 mm, vias 2 -> 4
- net /PROG_CLK: track 37.1 -> 36.4 mm
- net GND: track 32.1 -> 32.6 mm, vias 18 -> 17
- net /PA0: track 37.8 -> 38.4 mm
Other:
- board text added: "BOB v1.2"
- board text removed: "BOB v1.1"
- board text removed: "Doladit anténu - zkrátit připojení kondenzátorů. Navrhnout správně Microstrip nebo Grounded coplanar waveguide."

Commit message: bob 1.3
Parts:
- added R2: 4k7, Resistor_SMD:R_0805_2012Metric, F.Cu at (233.0, 60.5)
- added R5: 4k7, Resistor_SMD:R_0805_2012Metric, F.Cu at (233.0, 58.0)
- J3: footprint Connector_PinHeader_2.54mm:PinHeader_1x24_P2.54mm_Vertical -> Connector_PinHeader_2.54mm:PinHeader_1x26_P2.54mm_Vertical
- moved R1 10.4 mm to (230.5, 53.5), turned to 90 degrees
- moved C6 10.2 mm to (237.0, 63.0), turned to 0 degrees
- moved C5 7.21 mm to (233.0, 63.0)
- moved Y1 6.08 mm to (245.5, 62.0), turned to 90 degrees
- moved A1 6.00 mm to (245.0, 54.0)
- moved U1 6.00 mm to (239.5, 59.0)
- moved JP2 5.02 mm to (237.0, 54.0)
Connections:
- J3 pad 24: GND -> /PA7
- U1 pad 2: /RF_CLK -> /PA9
- U1 pad 3: /RF_DIO -> /PA7
- U3 pad 13: /RF_DIO -> /PA7
- U3 pad 19: /RF_CLK -> /PA9
Routing:
- net /PA9: track 0.00 -> 41.2 mm, vias 0 -> 2
- net /PA7: track 0.00 -> 40.0 mm, vias 0 -> 2
- net /RF_DIO: track 25.6 -> 0.00 mm, vias 2 -> 0
- net /RF_CLK: track 20.3 -> 0.00 mm, vias 2 -> 0
- net Net-(JP2-C): track 10.00 -> 7.09 mm
- net Net-(U1-XC0): track 5.67 -> 3.20 mm
- net GND: track 32.6 -> 30.5 mm, vias 17 -> 19
- net /PF1: track 26.0 -> 24.6 mm
- net Net-(U1-XC1): track 4.13 -> 5.28 mm
- net /PF3: track 25.2 -> 26.3 mm
- net /PF0: track 23.5 -> 22.8 mm
- net /PF4: track 13.1 -> 13.7 mm
- net +3V3: track 28.1 -> 27.6 mm, vias 7 -> 10
- net /~{RF_CS}: track 26.6 -> 27.1 mm
Other:
- board size 62 x 19 mm -> 68 x 19 mm
- board text added: "A7"
- board text added: "A9"
- board text added: "BOB v1.3"
- board text added: "RADIO"
- board text removed: "B4"
- board text removed: "B5"
- board text removed: "BOB v1.2"

Commit message: WIP
Other:
- board text added: "B4"
- board text added: "B5"

Commit message: Refactor code structure for improved readability and maintainability
Parts:
- removed JP2: I2C/SPI, Jumper:SolderJumper-3_P2.0mm_Open_TrianglePad1.0x1.5mm
- R3, R4: value 270R -> 330R
Connections:
- R1 pad 2: Net-(JP2-C) -> +3V3
Routing:
- net Net-(JP2-C): track 7.09 -> 0.00 mm
- net GND: track 30.5 -> 29.2 mm, vias 19 -> 18
- net +3V3: track 27.6 -> 28.1 mm
Other:
- board text added: "BOB v1.4"
- board text removed: "BOB v1.3"
