File: dongle/py32f403/board/dongle-py32f403.kicad_pcb (KiCad board)
At the start: 2 copper layers, 46.5 x 16 mm, 25 parts, among them J1 USB_A, U1 PAN2110P0AA, U2 PY32F403C1xT6, U4 XC6206P332MR, X1 SWD, Y1 16MHz, Y2 12MHz

Commit message: usb dongle v1.1
Connections:
- U2 pad 26: Net-(U2-PB13) -> unconnected-(U2-PB13-Pad26)
- U2 pad 27: Net-(U2-PB14) -> unconnected-(U2-PB14-Pad27)
- U2 pad 34: unconnected-(U2-PA13-Pad34) -> /SWD_IO
- U2 pad 37: unconnected-(U2-PA14-Pad37) -> /SWD_CLK
- X1 pad 1: Net-(U2-PB13) -> /SWD_IO
- X1 pad 3: Net-(U2-PB14) -> /SWD_CLK
Routing:
- net Net-(U2-PB14): track 7.92 -> 0.00 mm
- net /SWD_CLK: track 0.00 -> 4.54 mm, vias 0 -> 1
- net /SWD_IO: track 0.00 -> 4.10 mm
- net Net-(U2-PB13): track 3.55 -> 0.00 mm
- net GND: vias 57 -> 56
Other:
- board text added: "v1.1"
- board text removed: "v1.0"
Changed lines of the file:
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@@
 			(layers "*.Cu" "*.Mask")
 			(remove_unused_layers no)
-			(net "Net-(U2-PB13)")
+			(net "/SWD_IO")
 			(pinfunction "DIO_1")
 			(pintype "bidirectional")
@@
 			(layers "*.Cu" "*.Mask")
 			(remove_unused_layers no)
-			(net "Net-(U2-PB14)")
+			(net "/SWD_CLK")
 			(pinfunction "CLK_3")
 			(pintype "bidirectional")
@@
 			(layers "F.Cu" "F.Mask" "F.Paste")
 			(roundrect_rratio 0.25)
-			(net "Net-(U2-PB13)")
+			(net "unconnected-(U2-PB13-Pad26)")
 			(pinfunction "PB13_26")
-			(pintype "bidirectional")
+			(pintype "bidirectional+no_connect")
 		)
 		(pad "27" smd roundrect
@@
 			(layers "F.Cu" "F.Mask" "F.Paste")
 			(roundrect_rratio 0.25)
-			(net "Net-(U2-PB14)")
+			(net "unconnected-(U2-PB14-Pad27)")
 			(pinfunction "PB14_27")
-			(pintype "bidirectional")
+			(pintype "bidirectional+no_connect")
 		)
 		(pad "28" smd roundrect
@@
 			(layers "F.Cu" "F.Mask" "F.Paste")
 			(roundrect_rratio 0.25)
-			(net "unconnected-(U2-PA13-Pad34)")
+			(net "/SWD_IO")
 			(pinfunction "PA13_34")
-			(pintype "bidirectional+no_connect")
+			(pintype "bidirectional")
 		)
 		(pad "35" smd roundrect
@@
 			(layers "F.Cu" "F.Mask" "F.Paste")
 			(roundrect_rratio 0.25)
-			(net "unconnected-(U2-PA14-Pad37)")
+			(net "/SWD_CLK")
 			(pinfunction "PA14_37")
-			(pintype "bidirectional+no_connect")
+			(pintype "bidirectional")
 		)
 		(pad "38" smd roundrect
@@
 		(layer "Edge.Cuts")
 	)
-	(gr_text "v1.0"
+	(gr_text "v1.1"
 		(at 147 71 0)
 		(layer "B.SilkS")
@@
 	)
 	(via
-		(at 140.25 72.75)
-		(size 0.6)
-		(drill 0.3)
-		(layers "F.Cu" "B.Cu")
-		(free yes)
-		(net "GND")
-	)
-	(via
 		(at 163.9 68)
 		(size 0.6)
@@
 	)
 	(segment
-		(start 140.3375 65.75)
-		(end 139.21 65.75)
-		(width 0.2)
-		(layer "F.Cu")
-		(net "Net-(U2-PB13)")
-	)
-	(segment
-		(start 139.21 65.75)
-		(end 137.5 67.46)
-		(width 0.2)
-		(layer "F.Cu")
-		(net "Net-(U2-PB13)")
-	)
-	(segment
-		(start 140.3375 66.25)
-		(end 139.56759 66.25)
-		(width 0.2)
-		(layer "F.Cu")
-		(net "Net-(U2-PB14)")
-	)
-	(segment
-		(start 138.75 71.29)
-		(end 137.5 72.54)
-		(width 0.2)
-		(layer "F.Cu")
-		(net "Net-(U2-PB14)")
-	)
-	(segment
-		(start 139.56759 66.25)
-		(end 138.75 67.06759)
-		(width 0.2)
-		(layer "F.Cu")
-		(net "Net-(U2-PB14)")
-	)
-	(segment
-		(start 138.75 67.06759)
-		(end 138.75 71.29)
-		(width 0.2)
-		(layer "F.Cu")
-		(net "Net-(U2-PB14)")
-	)
-	(segment
 		(start 148.6625 67.75)
 		(end 149.841205 67.75)
@@
 	)
 	(segment
-		(start 135.475 68.5)
-		(end 134.545999 67.570999)
-		(width 0.2)
-		(layer "B.Cu")
-		(net "/USB_D-")
-	)
-	(segment
-		(start 134.545999 67.570999)
-		(end 134.16858 67.570999)
+		(start 137.060105 68.522)
+		(end 137.038105 68.5)
 		(width 0.2)
 		(layer "B.Cu")
@@
 	)
 	(segment
-		(start 137.038105 68.5)
-		(end 135.475 68.5)
+		(start 137.961895 68.5)
+		(end 137.939895 68.522)
 		(width 0.2)
 		(layer "B.Cu")
@@
 	)
 	(segment
-		(start 137.961895 68.5)
-		(end 137.939895 68.522)
+		(start 141.75 68.5)
+		(end 137.961895 68.5)
 		(width 0.2)
 		(layer "B.Cu")
@@
 	)
 	(segment
-		(start 137.060105 68.522)
-		(end 137.038105 68.5)
+		(start 135.097581 68.5)
+		(end 134.16858 67.570999)
 		(width 0.2)
 		(layer "B.Cu")
@@
 	)
 	(segment
-		(start 137.939895 68.522)
-		(end 137.060105 68.522)
+		(start 137.038105 68.5)
+		(end 135.097581 68.5)
 		(width 0.2)
 		(layer "B.Cu")
@@
 	)
 	(segment
-		(start 141.75 68.5)
-		(end 137.961895 68.5)
+		(start 137.939895 68.522)
+		(end 137.060105 68.522)
 		(width 0.2)
 		(layer "B.Cu")
@@
 		(net "Net-(D1-A)")
 	)
+	(segment
+		(start 139.25 69.75)
+		(end 140.3375 69.75)
+		(width 0.2)
+		(layer "F.Cu")
+		(net "/SWD_IO")
+	)
+	(segment
+		(start 137.5 68)
+		(end 139.25 69.75)
+		(width 0.2)
+		(layer "F.Cu")
+		(net "/SWD_IO")
+	)
+	(segment
+		(start 137.5 67.46)
+		(end 137.5 68)
+		(width 0.2)
+		(layer "F.Cu")
+		(net "/SWD_IO")
+	)
+	(segment
+		(start 141.5875 72)
+		(end 140.5 72)
+		(width 0.2)
+		(layer "F.Cu")
+		(net "/SWD_CLK")
+	)
+	(segment
+		(start 141.75 72.1625)
+		(end 141.5875 72)
+		(width 0.2)
+		(layer "F.Cu")
+		(net "/SWD_CLK")
+	)
+	(via
+		(at 140.5 72)
+		(size 0.6)
+		(drill 0.3)
+		(layers "F.Cu" "B.Cu")
+		(net "/SWD_CLK")
+	)
+	(segment
+		(start 140.5 72)
+		(end 139.96 72.54)
+		(width 0.2)
+		(layer "B.Cu")
+		(net "/SWD_CLK")
+	)
+	(segment
+		(start 139.96 72.54)
+		(end 137.5 72.54)
+		(width 0.2)
+		(layer "B.Cu")
+		(net "/SWD_CLK")
+	)
 	(zone
