File: dongle/py32f403/board/dongle-py32f403.kicad_sch (KiCad schematic)
At the start: 25 parts, among them J1 USB_A, U1 PAN2110P0AA, U2 PY32F403C1xT6, U4 XC6206P332MR, X1 SWD, Y1 16MHz, Y2 12MHz

Commit message: usb dongle v1.1
Connections:
- net at U2.26 (PB13): no longer X1.1 (DIO)
- net at U2.27 (PB14): no longer X1.3 (CLK)
- net SWD_IO: now reaches U2.34 (PA13)
- net SWD_IO: now also X1.1 (DIO)
- net SWD_CLK: now reaches U2.37 (PA14)
- net SWD_CLK: now also X1.3 (CLK)
Other:
- moved on the sheet: X1
Changed lines of the file:
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@@
-	)
-	(no_connect
-		(at 226.06 105.41)
 	)
 	(no_connect
@@
 	)
 	(no_connect
+		(at 226.06 125.73)
+	)
+	(no_connect
 		(at 177.8 105.41)
 	)
@@
 	)
 	(no_connect
-		(at 213.36 90.17)
-	)
-	(no_connect
 		(at 203.2 90.17)
 	)
@@
 	)
 	(no_connect
+		(at 226.06 123.19)
+	)
+	(no_connect
 		(at 205.74 138.43)
 	)
@@
 	(wire
 		(pts
+			(xy 214.63 88.9) (xy 213.36 90.17)
+		)
+		(stroke
+			(width 0)
+			(type default)
+		)
+	)
+	(wire
+		(pts
 			(xy 158.75 90.17) (xy 158.75 91.44)
 		)
@@
 	(wire
 		(pts
+			(xy 248.92 133.35) (xy 250.19 132.08)
+		)
+		(stroke
+			(width 0)
+			(type default)
+		)
+	)
+	(wire
+		(pts
 			(xy 191.77 139.7) (xy 190.5 138.43)
 		)
@@
 	(wire
 		(pts
+			(xy 248.92 135.89) (xy 250.19 134.62)
+		)
+		(stroke
+			(width 0)
+			(type default)
+		)
+	)
+	(wire
+		(pts
 			(xy 60.96 116.84) (xy 77.47 116.84)
 		)
@@
 		(pts
 			(xy 129.54 49.53) (xy 133.35 49.53)
+		)
+		(stroke
+			(width 0)
+			(type default)
+		)
+	)
+	(wire
+		(pts
+			(xy 227.33 106.68) (xy 226.06 105.41)
 		)
 		(stroke
@@
 		)
 	)
+	(label "SWD_IO"
+		(at 227.33 106.68 0)
+		(effects
+			(font
+				(size 1.27 1.27)
+			)
+			(justify left bottom)
+		)
+	)
+	(label "SWD_IO"
+		(at 248.92 135.89 180)
+		(effects
+			(font
+				(size 1.27 1.27)
+			)
+			(justify right bottom)
+		)
+	)
+	(label "SWD_CLK"
+		(at 214.63 88.9 90)
+		(effects
+			(font
+				(size 1.27 1.27)
+			)
+			(justify left bottom)
+		)
+	)
 	(label "USB_D+"
 		(at 227.33 109.22 0)
@@
 			)
 			(justify left bottom)
+		)
+	)
+	(label "SWD_CLK"
+		(at 248.92 133.35 180)
+		(effects
+			(font
+				(size 1.27 1.27)
+			)
+			(justify right bottom)
 		)
 	)
@@
 	(symbol
 		(lib_id "Drake:SWD")
-		(at 233.68 124.46 180)
+		(at 257.81 133.35 180)
 		(unit 1)
 		(body_style 1)
@@
 		(dnp no)
 		(property "Reference" "X1"
-			(at 234.315 132.08 0)
+			(at 258.445 140.97 0)
 			(show_name no)
 			(do_not_autoplace no)
@@
 		)
 		(property "Value" "SWD"
-			(at 234.315 129.54 0)
+			(at 258.445 138.43 0)
 			(show_name no)
 			(do_not_autoplace no)
@@
 		)
 		(property "Footprint" "Drake:SWD"
-			(at 233.68 115.57 0)
+			(at 257.81 124.46 0)
 			(hide yes)
 			(show_name no)
@@
 		)
 		(property "Datasheet" ""
-			(at 233.68 124.46 0)
+			(at 257.81 133.35 0)
 			(show_name no)
 			(do_not_autoplace no)
@@
 		)
 		(property "Description" ""
-			(at 233.68 124.46 0)
-			(hide yes)
-			(show_name no)
+			(at 257.81 133.35 0)
+			(hide yes)
+			(show_name no)
